Commit message: Add sprung bogie tracked chassis variant

File: urdf/tracked.urdf.xacro (robot description, xacro)
@@ -7,21 +7,11 @@
   <xacro:property name='body_clearance' value='0.17'/>
   <link name='base_link'>
-    <visual name='TRK-BASE-001_visual'>
-      <origin xyz='0 0 0.28' rpy='0 0 0'/>
-      <geometry><box size='0.7 0.4 0.22'/></geometry>
-    </visual>
-    <collision name='TRK-BASE-001_collision'>
-      <origin xyz='0 0 0.27' rpy='0 0 0'/>
-      <geometry><box size='0.68 0.37 0.2'/></geometry>
-    </collision>
-    <inertial>
-      <origin xyz='0 0 0.3' rpy='0 0 0'/>
-      <mass value='60.6'/>
-      <inertia ixx='1.0524200000000001' ixy='0' ixz='0' iyy='2.7189200000000002' iyz='0' izz='3.2824999999999993'/>
-    </inertial>
+    <visual name='TRK-BASE-001_visual'><origin xyz='0 0 0.28' rpy='0 0 0'/><geometry><box size='0.7 0.4 0.22'/></geometry></visual>
+    <collision name='TRK-BASE-001_collision'><origin xyz='0 0 0.27' rpy='0 0 0'/><geometry><box size='0.68 0.37 0.2'/></geometry></collision>
+    <inertial><origin xyz='0 0 0.3' rpy='0 0 0'/><mass value='60.6'/><inertia ixx='1.0524200000000001' ixy='0' ixz='0' iyy='2.7189200000000002' iyz='0' izz='3.2824999999999993'/></inertial>
   </link>
   <link name='left_wheel'><collision name='left_wheel_collision'><geometry><cylinder radius='0.12' length='0.09'/></geometry></collision></link>
+  <joint name='left_joint' type='continuous'><parent link='base_link'/><child link='left_wheel'/><origin xyz='0.0 0.26 0.12' rpy='1.57079632679 0 0'/><axis xyz='0 0 -1'/></joint>
   <link name='right_wheel'><collision name='right_wheel_collision'><geometry><cylinder radius='0.12' length='0.09'/></geometry></collision></link>
-  <joint name='left_joint' type='continuous'><parent link='base_link'/><child link='left_wheel'/><origin xyz='0.0 0.26 0.12' rpy='1.57079632679 0 0'/><axis xyz='0 0 -1'/></joint>
   <joint name='right_joint' type='continuous'><parent link='base_link'/><child link='right_wheel'/><origin xyz='0.0 -0.26 0.12' rpy='1.57079632679 0 0'/><axis xyz='0 0 -1'/></joint>
   <!-- Future CAD references: TRK-BASE-001, TRK-BELT-VIS-001, TRK-SUPPORT-SPHERE-001. Visual and collision geometry remain separate. -->

File: urdf/tracked_improved.urdf.xacro (robot description, xacro)
@@ -7,21 +7,11 @@
   <xacro:property name='body_clearance' value='0.25'/>
   <link name='base_link'>
-    <visual name='TRK2-BASE-001_visual'>
-      <origin xyz='0 0 0.35' rpy='0 0 0'/>
-      <geometry><box size='0.86 0.56 0.24'/></geometry>
-    </visual>
-    <collision name='TRK2-BASE-001_collision'>
-      <origin xyz='0 0 0.35' rpy='0 0 0'/>
-      <geometry><box size='0.78 0.48 0.2'/></geometry>
-    </collision>
-    <inertial>
-      <origin xyz='0 0 0.34' rpy='0 0 0'/>
-      <mass value='52.6'/>
-      <inertia ixx='1.6270933333333335' ixy='0' ixz='0' iyy='3.494393333333333' iyz='0' izz='4.616526666666666'/>
-    </inertial>
+    <visual name='TRK2-BASE-001_visual'><origin xyz='0 0 0.35' rpy='0 0 0'/><geometry><box size='0.86 0.56 0.24'/></geometry></visual>
+    <collision name='TRK2-BASE-001_collision'><origin xyz='0 0 0.35' rpy='0 0 0'/><geometry><box size='0.78 0.48 0.2'/></geometry></collision>
+    <inertial><origin xyz='0 0 0.34' rpy='0 0 0'/><mass value='52.6'/><inertia ixx='1.6270933333333335' ixy='0' ixz='0' iyy='3.494393333333333' iyz='0' izz='4.616526666666666'/></inertial>
   </link>
   <link name='left_wheel'><collision name='left_wheel_collision'><geometry><cylinder radius='0.18' length='0.13'/></geometry></collision></link>
+  <joint name='left_joint' type='continuous'><parent link='base_link'/><child link='left_wheel'/><origin xyz='0.16 0.35 0.18' rpy='1.57079632679 0 0'/><axis xyz='0 0 -1'/></joint>
   <link name='right_wheel'><collision name='right_wheel_collision'><geometry><cylinder radius='0.18' length='0.13'/></geometry></collision></link>
-  <joint name='left_joint' type='continuous'><parent link='base_link'/><child link='left_wheel'/><origin xyz='0.16 0.35 0.18' rpy='1.57079632679 0 0'/><axis xyz='0 0 -1'/></joint>
   <joint name='right_joint' type='continuous'><parent link='base_link'/><child link='right_wheel'/><origin xyz='0.16 -0.35 0.18' rpy='1.57079632679 0 0'/><axis xyz='0 0 -1'/></joint>
   <!-- Future CAD references: TRK2-BASE-001, TRK2-BELT-VIS-001, TRK2-REAR-SKID-001. Visual and collision geometry remain separate. -->
